File: uCurrent.brd (EAGLE design)
At the start: 49.6 x 74.6 mm, 48 parts, among them IC1 LMV321ILT, J1 CL2160B, J2 CL2160R, J3 930175101, J4 930175100, J5 B2B-PH-SM4-TB, SW1 L203011MS02Q, SW2 L203011MS02Q, U1 MAX4239AUT, U2 MAX4239AUT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

Commit message: Small updates and gerbers
Parts:
- moved R9 0.13 mm to (-10.9, 10.8)
Routing:
- net N$8: track 8.43 -> 10.9 mm
- net VGND: track 131.5 -> 132.9 mm
- net V+: track 112.5 -> 111.7 mm
- net N$11: track 18.1 -> 17.4 mm
- net IN_-VE: track 67.3 -> 66.8 mm
Other:
- board text added: "Max: 1250mA @ 3V Max: 2250mA @ 5V"
