File: uCurrent.sch (EAGLE design)
At the start: 48 parts, among them IC1 LMV321ILT, J1 CL2160B, J2 CL2160R, J3 930175101, J4 930175100, J5 B2B-PH-SM4-TB, SW1 L203011MS02Q, SW2 L203011MS02Q, U1 MAX4239AUT, U2 MAX4239AUT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

Commit message: Small updates and gerbers
Changed lines of the file:
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@@
 </class>
 <class number="1" name="Signal" width="0.25" drill="0">
+<clearance class="1" value="0.2"/>
 </class>
 <class number="2" name="LVDC" width="0.3" drill="0">
+<clearance class="2" value="0.2"/>
 </class>
 <class number="3" name="VOUT" width="0" drill="0">
@@
 <segment>
 <pinref part="U1" gate="G$1" pin="2"/>
-<wire x1="190.5" y1="162.56" x2="190.5" y2="157.48" width="0.1524" layer="91"/>
+<wire x1="190.5" y1="160.02" x2="190.5" y2="157.48" width="0.1524" layer="91"/>
 <wire x1="190.5" y1="157.48" x2="193.04" y2="157.48" width="0.1524" layer="91"/>
 <label x="193.04" y="157.48" size="1.778" layer="95"/>
@@
 <segment>
 <pinref part="U2" gate="G$1" pin="2"/>
-<wire x1="243.84" y1="162.56" x2="243.84" y2="157.48" width="0.1524" layer="91"/>
+<wire x1="243.84" y1="160.02" x2="243.84" y2="157.48" width="0.1524" layer="91"/>
 <wire x1="243.84" y1="157.48" x2="246.38" y2="157.48" width="0.1524" layer="91"/>
 <label x="246.38" y="157.48" size="1.778" layer="95"/>
